File: hardware/minirouter/MiniRouter.sch (EAGLE design)
At the start: 49 parts, among them J0 CON-MATENLOK, J1 AVR_PROG, J2 RJ45-8PTH, J3 RJ45-8PTH, J4 RJ45-8PTH, J5 RASPBERRY-PI_REV2, Q1 NMOS, Q2 NMOS, Q3 NMOS, U1 ATMEGA168, U2 AOZ1242SMD, U3 DS1307SO8, Y1 32.768kHz

Commit message: Checking in the latest schematics for the kickstarter
Parts:
- removed J0: CON-MATENLOK, pierre:CON-MATENLOK
- removed JP7: STAND-OFFTIGHT, SparkFun-Electromechanical:STAND-OFFTIGHT
- removed SJ1, SJ2: (no value), SparkFun-Passives:SOLDERJUMPER_2WAYPASTE1&2
- added F1: PTCSMD, SparkFun:PTCSMD
- added J6: 2.1MMJACKTHM, pierre:2.1MMJACKTHM
- renumbered CR1220 to J7
Connections:
- removed net RX0: J2.5, SJ1.3, U1.PD0(RXD)
- removed net U_RX: SJ1.1, U1.PB0(ICP)
- removed net U_TX: SJ2.1, U1.PB1(OC1A)
- new net N$5: C14.1, C15.1, C16.+, C4.+, F1.1, L1.2, R4.2
- new net RX3: J4.5, U1.PD7(AIN1)
- net 5V: now also F1.2; no longer C14.1, C15.1, C16.+, C4.+, L1.2, R4.2
- net GND: now also J6.RING, J6.RING_SW; no longer J0.2
- net RPI_RX: now also U1.PB0(ICP); no longer SJ1.2
- net RPI_TX: now also U1.PB1(OC1A); no longer SJ2.2
- net RX1: now also J2.5; no longer J3.5
- net RX2: now also J3.5, U1.PD5(T1); no longer J4.5, U1.PD4(XCK/T0)
- net TX: no longer SJ2.3
- net VIN: now also J6.TIP; no longer J0.1
Other:
- note added: "2"
- note removed: "1"
