File: hardware/router/Router.sch (EAGLE design)
At the start: 52 parts, among them J0 CON-MATENLOK, J1 AVR_PROG, J10 RJ45-8PTH, J11 RJ45-8PTH, J12 RJ45-8PTH, J13 RJ45-8PTH, J14 RJ45-8PTH, J15 RJ45-8PTH, J16 RJ45-8PTH, J17 RASPBERRYPI_BB, J18 RJ45-8PTH, J19 RJ45-8PTH, J2 RJ45-8PTH, J3 RJ45-8PTH, J4 RJ45-8PTH, J5 RJ45-8PTH, J6 RJ45-8PTH, J7 RJ45-8PTH, J8 RJ45-8PTH, J9 RJ45-8PTH, Q1 NMOS, Q2 NMOS, Q3 NMOS, U1 ATMEGA168, U3 DS1307SO8, Y1 32.768kHz

Commit message: Checking in the latest schematics for the kickstarter
Parts:
- removed BAT1: 3V, SparkFun-Electromechanical:BATTERY12PTH
- removed C1: 10u, SparkFun-Passives:CAP0603-CAP
- removed C4: 2.2u, SparkFun-Passives:CAP0603-CAP
- removed C8: 47u, SparkFun-Capacitors:CAP_POLD
- removed C9: 100n, SparkFun:CAP0603-CAP
- removed J0: CON-MATENLOK, pierre:CON-MATENLOK
- removed JP5, JP7, JP8, JP9: STAND-OFFTIGHT, SparkFun-Electromechanical:STAND-OFFTIGHT
- removed U2: (no value), SparkFun-PowerIC:V_REG_78XXSIDE
- added C10: 47u, SparkFun-Capacitors:CAP_POLD
- added C11, C12, C16: 100n, SparkFun:CAP0603-CAP
- added C13: 1u, SparkFun:CAP0603-CAP
- added C14, C17: 1n, SparkFun:CAP0603-CAP
- added C15: 10u, SparkFun-Capacitors:CAP1206
- added C18, C19: 22u, microbuilder:CAP_TANTALUMC/6032_REFLOW
- added D1: 30V3A, pierre:B330A
- added F1: PTCSMD, SparkFun-PowerIC:PTCSMD
- added J20: 3V, SparkFun-Electromechanical:BATTERY12PTH
- added J22: 5566-4, pierre:5566-4
- added L1: 6.8u, pierre:INDUCTORCR54
- added R4: 52.3k, SparkFun-Resistors:RESISTOR0603-RES
- added R5, R6: 10k, SparkFun-Resistors:RESISTOR0603-RES
- added TP1: GND, microbuilder:TESTPOINT
- added U4: AOZ1242SMD, pierre:AOZ1242SMD
- J10, J11, J12, J13, J14, J15, J16, J18, J19, J2, J3, J4, J5, J6, J7, J8: device SparkFun:RJ45-8PTH -> pierre:RJ45-8PTH; DIST (none) -> DigiKey; DIST_PN (none) -> 151-1099-ND; MFG (none) -> EDAC Inc; MFG_PN (none) -> A00-108-220-450
- J17: value RASPBERRYPI_BB -> RASPBERRY-PI_REV2; device pierre:RASPBERRYPI_BB -> pierre:RASPBERRY-PI_REV2
- J9: device SparkFun:RJ45-8PTH -> pierre:RJ45-8PTH
- R1, R3: value 300 -> 330
- R2: value 300 -> 200
Connections:
- net RX0 renamed RX8
- net RX7/MOSI renamed RX4/MOSI
- net RX8/MISO renamed RX12/MISO
- net RX9/SCK renamed RX5/SCK
- removed net RX12: J15.5, U1.PC0(ADC0)
- removed net RX4: J11.5, U1.PD6(AIN0)
- removed net RX5: J4.5, U1.PD7(AIN1)
- new net N$15: C14.1, R6.1
- new net N$16: C12.2, D1.C, L1.1, U4.LX
- new net N$2: R4.1, R5.2, U4.FB
- new net N$3: R6.2, U4.COMP
- new net N$5: C16.1, C17.1, C18.+, C19.+, F1.1, L1.2, R4.2
- new net N$7: C12.1, U4.BS
- new net N$8: C13.1, U4.VBIAS
- new net RX15: J16.5, U1.PC2(ADC2)
- new net RX7: J8.5, U1.PC1(ADC1)
- new net RX9: J10.5, U1.PD4(XCK/T0)
- net 3.3V: now also J17.3V3@1, J17.3V3@17; no longer J17.3.3V@1
- net 5V: now also F1.2, J17.5V@2, J17.5V@4; no longer C4.1, J17.5.0V@1, U2.OUT
- net BAT1+: now also J20.+; no longer BAT1.+
- net BLUE: now also J17.GPIO23; no longer J17.GPIO4
- net CE0: now also J17.GPIO8,SPI0_CE0; no longer J17.#SPI_CE0
- net CE1: now also J17.GPIO7,SPI0_CE1; no longer J17.#SPI_CE1
- net GND: now also C10.-, C11.2, C13.2, C14.2, C15.2, C16.2, C17.2, C18.-, C19.-, D1.A, J17.GND@14, J17.GND@20, J17.GND@25, J17.GND@6, J17.GND@9, J20.-, J22-1.S, J22-3.S, R5.1, TP1.P$1, U4.GND; no longer BAT1.-, C1.2, C4.2, C8.-, C9.2, J0.2, J17.GND, U2.GND
- net GREEN: now also J17.GPIO25; no longer J17.GPIO6
- net RED: now also J17.GPIO24; no longer J17.GPIO5
- net RPI_MISO: now also J17.GPIO9_MISO; no longer J17.SPI_MISO
- net RPI_MOSI: now also J17.GPIO10_MOSI; no longer J17.SPI_MOSI
- net RPI_RX: now also J17.GPIO15,UART0_RXD; no longer J17.RXD
- net RPI_SCL: now also J17.GPIO3,I2C0_SCL; no longer J17.SCL0
- net RPI_SCLK: now also J17.GPIO11_SCLK; no longer J17.SPI_SCLK
- net RPI_SDA: now also J17.GPIO2,I2C0_SDA; no longer J17.SDA0
- net RPI_TX: now also J17.GPIO14,UART0_TXD; no longer J17.TXD
- net RX10: now also J11.5, U1.PD6(AIN0); no longer J14.5, U1.PB6(XTAL1/TOSC1)
- net RX11: now also J12.5, U1.PB2(SS/OC1B); no longer J7.5, U1.PB7(XTAL2/TOSC2)
- net RX13: now also J14.5, U1.PB6(XTAL1/TOSC1); no longer J8.5, U1.PC1(ADC1)
- net RX14: now also J15.5, U1.PC0(ADC0); no longer J16.5, U1.PC2(ADC2)
- net RX2: now also J3.5, U1.PD5(T1); no longer J10.5, U1.PD4(XCK/T0)
- net RX3: now also J4.5, U1.PD7(AIN1); no longer J3.5, U1.PD5(T1)
- net RX6: now also J7.5, U1.PB7(XTAL2/TOSC2); no longer J12.5, U1.PB2(SS/OC1B)
- net VIN: now also C10.+, C11.1, C15.1, J22-2.S, J22-4.S, U4.EN, U4.VIN; no longer C1.1, C8.+, C9.1, J0.1, U2.IN
Other:
- note added: "2"
- note added: "24V 3A"
- note added: "5V 3A Out"
- note added: "Accessory Port 2"
- note removed: "1.1"
- note removed: "5V 2A Out"
- note removed: "Accessory Port 0"
- moved on the sheet: C2, C3, C5, C6, C7, R9, U1, U3, Y1
